Commit message: add steering angle visualization to robot model; make putnam launch file working again

File: src/launch/racing_lmpc_launch/config/urdf/iac_car/av21.urdf (robot description, URDF)
Before this commit: robot AV 21, 41 links, 40 joints
Links:
- link model: geometry visual mesh filename=package://racing_lmpc_launch/config/urdf/iac_car/visual/il1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 scale=0.01 0.01 0.01
- link tyre_fl: geometry visual mesh filename=package://racing_lmpc_launch/config/urdf/iac_car/visual/il1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 scale=0.01 0.01 0.01
- link tyre_fr: geometry visual mesh filename=package://racing_lmpc_launch/config/urdf/iac_car/visual/il1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 scale=0.01 0.01 0.01
- link tyre_rl: geometry visual mesh filename=package://racing_lmpc_launch/config/urdf/iac_car/visual/il1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 scale=0.01 0.01 0.01
- link tyre_rr: geometry visual mesh filename=package://racing_lmpc_launch/config/urdf/iac_car/visual/il1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 scale=0.01 0.01 0.01
Joints:
- joint fl_tyre_joint: axis (none) -> 0 0 1; limit (none) -> lower=-0.523599 upper=0.523599 effort=1000 velocity=1; type fixed -> revolute
- joint fr_tyre_joint: axis (none) -> 0 0 1; limit (none) -> lower=-0.523599 upper=0.523599 effort=1000 velocity=1; type fixed -> revolute
- joint model_joint: origin xyz=1.725 0.0 -0.31 rpy=1.5708 0.0 1.5708 -> xyz=1.725 0.0 -0.31 rpy=0 0.0 1.5708

Commit message: undo body urdf rotate; just change foxglove 3d pannel setting: mesh to be z axis up

File: src/launch/racing_lmpc_launch/config/urdf/iac_car/av21.urdf (robot description, URDF)
Before this commit: robot AV 21, 41 links, 40 joints
Joints:
- joint model_joint: origin xyz=1.725 0.0 -0.31 rpy=0 0.0 1.5708 -> xyz=1.725 0.0 -0.31 rpy=1.5708 0.0 1.5708

Commit message: wip visualize wheel spin

File: src/launch/racing_lmpc_launch/config/urdf/iac_car/av21.urdf (robot description, URDF)
Before this commit: robot AV 21, 41 links, 40 joints
Links:
- added link tyre_fl_rotate
- added link tyre_fr_rotate
- added link tyre_rl_rotate
- added link tyre_rr_rotate
Joints:
- added joint fl_tyre_rotate_joint: type revolute, parent tyre_fl_rotate, child tyre_fl, origin xyz=0.0 0.0 0.0 rpy=0 0 0, axis 1 0 0, limit lower=-3.15 upper=3.15 effort=1000 velocity=100
- added joint fr_tyre_rotate_joint: type revolute, parent tyre_fr_rotate, child tyre_fr, origin xyz=0.0 0.0 0.0 rpy=0 0 0, axis 1 0 0, limit lower=-3.15 upper=3.15 effort=1000 velocity=100
- added joint rl_tyre_rotate_joint: type revolute, parent tyre_rl_rotate, child tyre_rl, origin xyz=0.0 0.0 0.0 rpy=0 0 0, axis 1 0 0, limit lower=-3.15 upper=3.15 effort=1000 velocity=100
- added joint rr_tyre_rotate_joint: type revolute, parent tyre_rr_rotate, child tyre_rr, origin xyz=0.0 0.0 0.0 rpy=0 0 0, axis 1 0 0, limit lower=-3.15 upper=3.15 effort=1000 velocity=100
- joint fl_tyre_joint: child tyre_fl -> tyre_fl_rotate
- joint fr_tyre_joint: child tyre_fr -> tyre_fr_rotate
- joint rl_tyre_joint: child tyre_rl -> tyre_rl_rotate
- joint rr_tyre_joint: child tyre_rr -> tyre_rr_rotate
